File: DA_02_0V1_F03_FC.kicad_pcb (KiCad board)
At the start: 2 copper layers, 33 x 37.5 mm, 89 parts, among them P3 2x2-SMD_PAD, P4 2x2-SMD_PAD, P5 2x2-SMD_PAD, P6 2x2-SMD_PAD, P7 2x2-SMD_PAD, P8 2x2-SMD_PAD, P9 2x2-SMD_PAD, Q1 SQ2310ES-T1_GE3, Q2 SQ2310ES-T1_GE3, Q3 SQ2310ES-T1_GE3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

Commit message: Production File
Other:
- board text added: "JLCJLCJLCJLC"
